Commit message: moveit urdf 수정전

File: urdf/arm1_URDF.urdf (robot description, URDF)
Before this commit: robot arm1_URDF, 9 links, 9 joints
Links:
- added link world
- link G_13: geometry collision mesh filename=package://final_project/meshes/G_13.stl scale=0.001 0.001 0.001; visual mesh filename=package://final_project/meshes/G_13.stl scale=0.001 0.001 0.001
- link G_2: geometry collision mesh filename=package://final_project/meshes/G_2.stl scale=0.001 0.001 0.001; visual mesh filename=package://final_project/meshes/G_2.stl scale=0.001 0.001 0.001
- link G_25: geometry collision mesh filename=package://final_project/meshes/G_25.stl scale=0.001 0.001 0.001; visual mesh filename=package://final_project/meshes/G_25.stl scale=0.001 0.001 0.001
- link G_27: geometry collision mesh filename=package://final_project/meshes/G_27.stl scale=0.001 0.001 0.001; visual mesh filename=package://final_project/meshes/G_27.stl scale=0.001 0.001 0.001
- link G_28: geometry collision mesh filename=package://final_project/meshes/G_28.stl scale=0.001 0.001 0.001; visual mesh filename=package://final_project/meshes/G_28.stl scale=0.001 0.001 0.001
- link G_4: geometry collision mesh filename=package://final_project/meshes/G_4.stl scale=0.001 0.001 0.001; visual mesh filename=package://final_project/meshes/G_4.stl scale=0.001 0.001 0.001
- link G_5: geometry collision mesh filename=package://final_project/meshes/G_5.stl scale=0.001 0.001 0.001; visual mesh filename=package://final_project/meshes/G_5.stl scale=0.001 0.001 0.001
- link G_7: geometry collision mesh filename=package://final_project/meshes/G_7.stl scale=0.001 0.001 0.001; visual mesh filename=package://final_project/meshes/G_7.stl scale=0.001 0.001 0.001
- link base: geometry collision mesh filename=package://final_project/meshes/base.stl scale=0.001 0.001 0.001; visual mesh filename=package://final_project/meshes/base.stl scale=0.001 0.001 0.001
Joints:
- removed joint 강체-17
- removed joint 강체-18
- removed joint 회전-10
- removed joint 회전-11
- removed joint 회전-12
- removed joint 회전-13
- removed joint 회전-14
- removed joint 회전-15
- removed joint 회전-16
- added joint fixed_18: type fixed, parent base, child G_2, origin xyz=0.09099999979871715 -3.750249421563545e-09 1.0266500027019778 rpy=8.673617379883954e-19 1.3065901218165487e-62 1.5777218104420236e-30
- added joint joint_10: type continuous, parent G_2, child G_4, origin xyz=0.11955 0.040374999999999994 -0.051650000000000064 rpy=-3.5113466634615537e-31 -0.0 -2.3738919364399067e-66, axis 1.0 0.0 -2.465190328815662e-32
- added joint joint_11: type continuous, parent G_2, child G_5, origin xyz=-3.552713678800501e-17 0.051650000000000064 0.019750000000000004 rpy=1.5707963267948966 4.463542775542222e-47 5.605193857299268e-45, axis 0.0 1.0 4.4755935958520466e-31
- added joint joint_12: type continuous, parent G_5, child G_7, origin xyz=-0.0001249999999999929 -0.039 -0.19194999999999993 rpy=-1.8487926954202153e-15 -1.5707963267948966 0, axis 1.0 5.827954054064347e-31 -1.2351231148954849e-14
- added joint joint_13: type continuous, parent G_7, child G_25, origin xyz=-0.05755000000000066 7.382983113757291e-17 -0.04 rpy=4.70462019996466e-32 1.5707963267948841 0, axis 1.0 0.0 2.891008291347084e-31
- added joint joint_14: type continuous, parent G_27, child G_28, origin xyz=0.017250000000000015 0.0 -0.05025000000000006 rpy=-6.312213884124065e-64 4.930380657631324e-32 1.1347551481098548e-32, axis 4.930380657631324e-32 0.0 1.0
- added joint joint_15: type continuous, parent G_25, child G_27, origin xyz=-0.04 0.0 -0.24949997999999995 rpy=-7.591481487369757e-65 -3.9686267332812115e-32 6.6682750465799775e-34, axis 9.860761315262648e-32 0.0 1.0
- added joint joint_16: type continuous, parent G_28, child G_13, origin xyz=-0.004250000000000007 -0.02075 -0.05074999999999996 rpy=-1.8856650730814692e-65 4.930380657631324e-32 -2.613319425339874e-33, axis 0.0 0.0 1.0
- added joint world_to_base: type fixed, parent world, child base, origin xyz=0 0 0 rpy=0 0 0
